File: BigClock.brd (EAGLE design)
At the start: 193 x 100 mm, 50 parts, among them IC12 LM317MBT, IC16 7805, IC5 74LS47N, IC6 74LS47N, IC7 74LS47N, IC8 74LS47N

Commit message: Displays routed on schematics
Parts:
- removed DIS1, DIS2, DIS3, DIS4: SA23-11, display-kingbright:SX23-XX
- removed IC5, IC6, IC7, IC8: 74LS47N, 74xx-eu:DIL16
- removed R40, R41, R42, R43, R44, R45, R46, R47, R48, R49, R50, R51, R52, R53, R54, R55, R56, R57, R58, R59, R60, R61, R62, R63, R64, R65, R67: 330R, rcl:0204/5
- removed R66: (no value), rcl:0204/5
- added IC1: PIC16F628P, microchip:DIL18
- added IC2: (no value), uln-udn:DIL18
- added R1, R2, R3, R4, R5, R6, R7, R8: 330R, rcl:0204/5
- added U$1, U$2, U$3, U$4: SC23-11, display-kingbright:SX23-XX
Connections:
- removed net N$10: DIS1.2, R42.1
- removed net N$100: IC6.10, R57.2
- removed net N$101: IC6.11, R58.2
- removed net N$102: IC6.12, R59.2
- removed net N$103: IC6.13, R60.2
- removed net N$104: DIS4.10, R61.1
- removed net N$105: DIS4.9, R62.1
- removed net N$106: DIS4.2, R63.1
- removed net N$107: DIS4.3, R64.1
- removed net N$108: DIS4.4, R65.1
- removed net N$109: DIS4.6, R66.1
- removed net N$11: IC7.10, R43.2
- removed net N$110: DIS4.7, R67.1
- removed net N$111: IC8.14, R61.2
- removed net N$112: IC8.15, R62.2
- removed net N$113: IC8.9, R63.2
- removed net N$114: IC8.10, R64.2
- removed net N$115: IC8.11, R65.2
- removed net N$116: IC8.12, R66.2
- removed net N$117: IC8.13, R67.2
- removed net N$24: DIS1.3, R43.1
- removed net N$25: IC7.11, R44.2
- removed net N$26: DIS1.4, R44.1
- removed net N$27: IC7.12, R45.2
- removed net N$28: DIS1.6, R45.1
- removed net N$29: IC7.13, R46.2
- removed net N$30: DIS1.7, R46.1
- removed net N$38: IC5.14, R47.2
- removed net N$39: IC5.15, R48.2
- removed net N$40: IC5.9, R49.2
- removed net N$41: IC5.10, R50.2
- removed net N$42: IC5.11, R51.2
- removed net N$43: IC5.12, R52.2
- removed net N$44: IC5.13, R53.2
- removed net N$6: DIS1.10, R40.1
- removed net N$7: IC7.15, R41.2
- removed net N$8: DIS1.9, R41.1
- removed net N$88: DIS3.10, R54.1
- removed net N$9: IC7.9, R42.2
- removed net N$91: DIS3.9, R55.1
- removed net N$92: DIS3.2, R56.1
- removed net N$93: DIS3.3, R57.1
- removed net N$94: DIS3.4, R58.1
- removed net N$95: DIS3.6, R59.1
- removed net N$96: DIS3.7, R60.1
- removed net N$97: IC6.14, R54.2
- removed net N$98: IC6.15, R55.2
- removed net N$99: IC6.9, R56.2
- new net DISP_DP: IC1.6, R8.2
- new net DIS_A: IC1.13, R1.2
- new net DIS_B: IC1.12, R2.2
- new net DIS_C: IC1.11, R3.2
- new net DIS_C1: IC2.18, U$1.1, U$1.5
- new net DIS_C2: IC2.17, U$2.1, U$2.5
- new net DIS_C3: IC2.16, U$3.1, U$3.5
- new net DIS_C4: IC2.15, U$4.1, U$4.5
- new net DIS_D: IC1.10, R4.2
- new net DIS_E: IC1.9, R5.2
- new net DIS_F: IC1.8, R6.2
- new net DIS_G: IC1.7, R7.2
- new net N$1: R8.1, U$1.8, U$2.8, U$3.8, U$4.8
- new net N$2: IC1.2, IC2.1
- new net N$3: IC1.1, IC2.2
- new net N$4: IC1.18, IC2.3
- net +12V: no longer DIS1.1, DIS1.5, DIS2.1, DIS2.5, DIS3.1, DIS3.5, DIS4.1, DIS4.5
- net +5V: no longer IC5.16, IC5.3, IC5.4, IC5.5, IC6.16, IC6.3, IC6.4, IC6.5, IC7.16, IC7.3, IC7.4, IC8.16, IC8.3, IC8.4, IC8.5
- net GND: now also IC1.5, IC2.9; no longer IC5.8, IC6.8, IC7.5, IC7.8, IC8.8
- net N$31: now also R7.1, U$1.10, U$2.10, U$3.10, U$4.10; no longer DIS2.10, R47.1
- net N$32: now also R6.1, U$1.9, U$2.9, U$3.9, U$4.9; no longer DIS2.9, R48.1
- net N$33: now also R5.1, U$1.2, U$2.2, U$3.2, U$4.2; no longer DIS2.2, R49.1
- net N$34: now also R4.1, U$1.3, U$2.3, U$3.3, U$4.3; no longer DIS2.3, R50.1
- net N$35: now also R3.1, U$1.4, U$2.4, U$3.4, U$4.4; no longer DIS2.4, R51.1
- net N$36: now also R2.1, U$1.6, U$2.6, U$3.6, U$4.6; no longer DIS2.6, R52.1
- net N$37: now also R1.1, U$1.7, U$2.7, U$3.7, U$4.7; no longer DIS2.7, R53.1
- net N$5: now also IC1.17, IC2.4; no longer IC7.14, R40.2
- net VCC: now also IC1.14
Routing:
- net N$31: track 14.0 -> 190.6 mm, vias 0 -> 4
- net N$32: track 13.4 -> 180.1 mm, vias 0 -> 4
- net N$33: track 27.9 -> 185.2 mm, vias 0 -> 6
- net N$34: track 27.9 -> 175.1 mm, vias 0 -> 6
- net N$37: track 24.8 -> 170.2 mm, vias 0 -> 4
- net N$35: track 27.9 -> 164.5 mm, vias 0 -> 4
- net N$36: track 30.8 -> 159.9 mm, vias 0 -> 4
- net GND: track 86.1 -> 0.00 mm
- net N$94: track 43.2 -> 0.00 mm
- net N$93: track 43.2 -> 0.00 mm
- net N$92: track 43.2 -> 0.00 mm
- net N$109: track 41.8 -> 0.00 mm
- net N$95: track 35.3 -> 0.00 mm
- net N$108: track 35.1 -> 0.00 mm
- net N$107: track 34.0 -> 0.00 mm
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Other:
- board size 193 x 100 mm -> 207 x 100 mm
- board text removed: "REV 1.0"
